File: rfd77101-ih-cooker.kicad_pcb (KiCad board)
At the start: 2 copper layers, 27.9 x 32.4 mm, 27 parts, among them J1 Conn_01x02, J2 Conn_input, J3 Conn_01x07, J4 Conn_output, Q1 BSS138, Q2 BSS138, U1 RFD77101, U2 MAX31855KASA, U3 AP2204K-3.0, U4 MCP6002-xMC

Commit message: minors
Parts:
- added G***: LOGO, Logo:logo_didee, B.Cu at (154.9, 101.0)
- J1: footprint TerminalBlock_RND:TerminalBlock_RND_205-00241_1x02_P10.16mm_Horizontal -> TerminalBlock_RND:TerminalBlock_RND_205-00067_1x02_P7.50mm_Horizontal
- moved R8 8.62 mm to (145.0, 110.5)
- moved R9 4.95 mm to (146.2, 113.5), turned to 270 degrees
- moved J1 2.65 mm to (151.3, 118.0)
- moved R7 2.37 mm to (142.7, 116.4)
- moved R6 2.24 mm to (142.7, 118.0)
- moved R10 1.92 mm to (145.6, 116.4)
- moved C6 1.85 mm to (145.7, 118.0)
- moved U4 0.25 mm to (144.1, 113.4)
Connections:
- U1 pad 17: (no net) -> /LV_I
- U1 pad 18: (no net) -> /LV_O
- U1 pad 22: (no net) -> /LV_Power_I
- U1 pad 24: /LV_Power_I -> (no net)
- U1 pad 27: (no net) -> /MISO
- U1 pad 28: /LV_O -> /~SS
- U1 pad 29: /LV_I -> /SCK
- U2 pad 5: (no net) -> /SCK
- U2 pad 6: (no net) -> /~SS
- U2 pad 7: (no net) -> /MISO
Routing:
- net GND: track 51.4 -> 79.0 mm, vias 0 -> 8
- net Net-(R10-Pad2): track 0.00 -> 23.6 mm, vias 0 -> 2
- net +5V: track 20.1 -> 41.4 mm
- net /LV_Power_I: track 0.00 -> 20.7 mm, vias 0 -> 2
- net /Power_O: track 0.00 -> 13.6 mm
- net /LV_I: track 1.57 -> 13.7 mm, vias 0 -> 2
- net VDD: track 36.5 -> 44.3 mm
- net /Power_I: track 0.00 -> 6.91 mm
- net /LV_O: track 1.53 -> 6.38 mm
- net Net-(R6-Pad1): track 0.00 -> 4.07 mm
- net /LV_Power_O: track 0.00 -> 3.28 mm
- net Net-(R8-Pad1): track 0.00 -> 3.15 mm
- net /SCK: track 0.00 -> 3.12 mm
- net /MISO: track 0.00 -> 2.99 mm
- net /~SS: track 0.00 -> 2.80 mm
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- added copper zone on B.Cu, net GND
- added copper zone on F.Cu, net Net-(C1-Pad1)
- added copper zone on F.Cu, net Net-(C1-Pad2)
- added copper zone on F.Cu, net VDD
- removed copper zone on F.Cu, net GND
Other:
- board size 27.9 x 32.4 mm -> 29 x 35 mm
- board text added: "IN"
- board text added: "OUT"
