File: rfd77101-ih-cooker.sch (KiCad schematic (older format))
At the start: 27 parts, among them J1 Conn_01x02, J2 Conn_input, J3 Conn_01x07, J4 Conn_output, Q1 BSS138, Q2 BSS138, U1 RFD77101, U2 MAX31855KASA, U3 AP2204K-3.0, U4 MCP6002-xMC

Commit message: minors
Parts:
- J1: footprint TerminalBlock_RND:TerminalBlock_RND_205-00241_1x02_P10.16mm_Horizontal -> TerminalBlock_RND:TerminalBlock_RND_205-00067_1x02_P7.50mm_Horizontal
Changed lines of the file:
@@
 F 0 "J1" H 3270 3775 50  0000 C CNN
 F 1 "Conn_01x02" H 3270 3866 50  0000 C CNN
-F 2 "TerminalBlock_RND:TerminalBlock_RND_205-00241_1x02_P10.16mm_Horizontal" H 3350 4100 50  0001 C CNN
+F 2 "TerminalBlock_RND:TerminalBlock_RND_205-00067_1x02_P7.50mm_Horizontal" H 3350 4100 50  0001 C CNN
 F 3 "~" H 3350 4100 50  0001 C CNN
 	1    3350 4100
@@
 Text Label 2150 6600 2    50   ~ 0
 LV_I
-Text Label 7350 3950 2    50   ~ 0
+Text Label 7350 3550 2    50   ~ 0
 LV_O
-Text Label 7350 4050 2    50   ~ 0
+Text Label 7350 3750 2    50   ~ 0
 LV_I
 $Comp
@@
 Text Label 6400 7000 0    50   ~ 0
 LV_Power_I
-Text Label 7350 2850 2    50   ~ 0
+Text Label 7350 2950 2    50   ~ 0
 LV_Power_I
 Text Label 9100 3550 0    50   ~ 0
 LV_Power_O
+Text Label 7350 4050 2    50   ~ 0
+SCK
+Text Label 7350 3950 2    50   ~ 0
+~SS
+Text Label 7350 3650 2    50   ~ 0
+MISO
 $EndSCHEMATC
